File: Projects/LEDStrip/PCB/KiCad/peripheralspower.kicad_sch (KiCad schematic)
At the start: 6 parts, among them U3 LM2596S-5

Commit message: pcb changes
Parts:
- removed CIN1, CIN2: 330uF, Capacitor_Tantalum_SMD:CP_EIA-7360-38_Kemet-E, symbol Device:C_Polarized_Small
- removed COUT1: 220uF, Capacitor_Tantalum_SMD:CP_EIA-3216-18_Kemet-A, symbol Device:C_Polarized_Small
- removed D3: SK32, Diode_SMD:D_SMA, symbol Device:D_Schottky
- removed L1: 3uH, Inductor_SMD:L_Coilcraft_XAL7070-XXX, symbol Device:L_Small
- removed U3: LM2596S-5, Package_TO_SOT_SMD:TO-263-5_TabPin3, symbol Regulator_Switching:LM2596S-5
- added CIN3, CIN4: 330uF, Capacitor_Tantalum_SMD:CP_EIA-7360-38_Kemet-E, symbol Device:C_Polarized_Small
- added COUT2: 220uF, Capacitor_Tantalum_SMD:CP_EIA-3216-18_Kemet-A, symbol Device:C_Polarized_Small
- added D7: SK32, Diode_SMD:D_SMA, symbol Device:D_Schottky
- added L2: 3uH, Inductor_SMD:L_Coilcraft_XAL7070-XXX, symbol Device:L_Small
- added U5: LM2596S-5, Package_TO_SOT_SMD:TO-263-5_TabPin3, symbol Regulator_Switching:LM2596S-5
Connections:
- net VDD_12V: now also CIN3.1, CIN4.1, U5.1 (VIN)
- net VDD_5V: now also COUT2.1, L2.2, U5.4 (FB)
- new net: CIN3.2, CIN4.2
- new net: D7.1 (K), L2.1, U5.2 (OUT)
