File: Projects/LEDStrip/PCB/KiCad/LEDStrip.kicad_sch (KiCad schematic)
At the start: 41 parts, among them J1 USB_C_Receptacle_USB2.0_16P, J2 RGB LED, J3 LED ADDR, J4 LED MATRIX, J5 MAX9814, J6 SSD1306, J7 TFT, Q1 IRFML8244, Q2 IRFML8244, Q3 IRFML8244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

Commit message: pcb changes
Parts:
- removed J2: RGB LED, Connector_Molex:Molex_KK-254_AE-6410-04A_1x04_P2.54mm_Vertical, symbol Connector_Generic:Conn_01x04
- removed J3: LED ADDR, symbol Connector_Generic:Conn_01x03
- removed J4: LED MATRIX, symbol Connector_Generic:Conn_01x05
- removed J5: MAX9814, symbol Connector_Generic:Conn_01x05
- added H1, H2, H3, H4: Hole_Pad, MountingHole:MountingHole_3.2mm_M3_ISO7380_Pad, symbol Mechanical:MountingHole_Pad
- added J2: RGB LED, Connector_JST:JST_SH_SM04B-SRSS-TB_1x04-1MP_P1.00mm_Horizontal, symbol Connector_Generic_MountingPin:Conn_01x04_MountingPin
- added J3: LED ADDR, Connector_JST:JST_SH_SM03B-SRSS-TB_1x03-1MP_P1.00mm_Horizontal, symbol Connector_Generic_MountingPin:Conn_01x03_MountingPin
- added J4: LED MATRIX, Connector_JST:JST_SH_SM05B-SRSS-TB_1x05-1MP_P1.00mm_Horizontal, symbol Connector_Generic_MountingPin:Conn_01x05_MountingPin
- added J5: Barrel Jack, Connector_BarrelJack:BarrelJack_Kycon_KLDX-0202-xC_Horizontal, symbol Connector:Barrel_Jack_Switch_Pin3Ring
- J1: value USB_C_Receptacle_USB2.0_16P -> USB_C
- J6: footprint Connector_Molex:Molex_KK-254_AE-6410-04A_1x04_P2.54mm_Vertical -> Connector_PinHeader_2.54mm:PinHeader_1x04_P2.54mm_Vertical
- J7: footprint (none) -> Connector_PinHeader_2.54mm:PinHeader_1x08_P2.54mm_Vertical
- JP1: footprint (none) -> Jumper:SolderJumper-3_P1.3mm_Open_RoundedPad1.0x1.5mm_NumberLabels
- Q1, Q2, Q3: footprint Package_DirectFET:DirectFET_SB -> Package_TO_SOT_SMD:SOT-23
Connections:
- net LED_B: now also J2.4 (Pin_4)
- net LED_G: now also J2.2 (Pin_2)
- net LED_R: now also J2.3 (Pin_3)
- net MAT_CLK: now also J4.1 (Pin_1)
- net MAT_CS: now also J4.2 (Pin_2)
- net MAT_DIN: now also J4.3 (Pin_3)
- net PER_5V: now also J3.1 (Pin_1), J4.5 (Pin_5)
- net VCC_12V: now also J2.1 (Pin_1), J5.1
- net at R9.2: now also J3.2 (Pin_2)
- new net: H1.1, H2.1, H3.1, H4.1
- no-connect marks 2 -> 3
Other:
- sheet Peripherals Power: file boardvoltage.kicad_sch -> peripheralspower.kicad_sch
- note added: "MAX9814 Amplified Microphone"
- note removed: "MAX9814 Microphone"

Commit message: pcb changes
Parts:
- removed SW3: CMD BTN, Connector_Hirose:Hirose_DF13-04P-1.25DSA_1x04_P1.25mm_Vertical, symbol Switch:SW_Push_LED
- added R15: 330, Resistor_SMD:R_0603_1608Metric, symbol Device:R
- added R16: 1k, Resistor_SMD:R_0603_1608Metric, symbol Device:R
- added SW3: CMD BTN, IguanaLibrary:SW_RGB_JST_SH, symbol Iguana_Library:RGB_SWITCH_COMCATH
- R11: value 1k -> 330
Connections:
- net CMD_BTN: now also R16.2, SW3.NO1; no longer R11.2
- net ESP_3V3: now also SW3.C1
- net RGB_B: now also R15.2
- net RGB_G: now also R11.2
- net RGB_R: now also R10.2
- net at R11.1: now also SW3.G; no longer R10.1
- new net: R16.1, SW3.C2
- new net: R15.1, SW3.B
- new net: R10.1, SW3.R
Other:
- note added: "Command Button"
- note added: "Holes"
- moved on the sheet: J6

Commit message: PCB changes - almost complete, still needs copper fill
Parts:
- removed J3: LED ADDR, Connector_JST:JST_SH_SM03B-SRSS-TB_1x03-1MP_P1.00mm_Horizontal, symbol Connector_Generic_MountingPin:Conn_01x03_MountingPin
- removed R9: 330, Resistor_SMD:R_0603_1608Metric, symbol Device:R
- added J3: LED ADDR, Connector_JST:JST_EH_S4B-EH_1x04_P2.50mm_Horizontal, symbol Connector_Generic:Conn_01x04
Connections:
- net PER_5V is gone; now on net VCC_5V: J4.5 (Pin_5)
- net LED_ADDR: now also J3.2 (Pin_2)
- net VCC_12V: now also J3.1 (Pin_1)
- new net: J3.3 (Pin_3), J3.4 (Pin_4)
Other:
- removed sheet Peripherals Power

Commit message: pcb final
Connections:
- net GND: now reaches U2.1 (GND), U2.40 (GND), U2.41 (GND)
Changed lines of the file:
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@@
+		)
+	)
+	(global_label "GND"
+		(shape input)
+		(at 146.05 100.33 0)
+		(fields_autoplaced yes)
+		(effects
+			(font
+				(size 1.27 1.27)
+			)
+			(justify left)
+		)
+		(property "Intersheetrefs" "${INTERSHEET_REFS}"
+			(at 152.9057 100.33 0)
+			(effects
+				(font
+					(size 1.27 1.27)
+				)
+				(justify left)
+				(hide yes)
+			)
 		)
 	)

Commit message: checks and finishing
Connections:
- net VDD_EQ is gone; now on net VCC_5V: C10.1, R5.2, U1.1 (VDD)
- net ESP_3V3 renamed VCC_3V3
- net GND: no longer names the net of U2.1 (GND), U2.40 (GND), U2.41 (GND)
- no-connect marks 3 -> 21
