File: Projects/LEDStrip/PCB/KiCad/espbuttons.kicad_sch (KiCad schematic)
At the start: 3 parts, among them SW2 SW_DIP_x01

Commit message: checks and finishing
Connections:
- net ESP_3V3 renamed VCC_3V3
Changed lines of the file:
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@@
 		)
 	)
-	(global_label "ESP_3V3"
+	(global_label "VCC_3V3"
 		(shape input)
 		(at 45.72 20.32 0)
