File: Projects/LEDStrip/PCB/KiCad/max9814.kicad_sch (KiCad schematic)
At the start: 12 parts, among them U6 MAX9814

Commit message: pcb changes
Parts:
- removed MK1: Microphone_Condenser, symbol Device:Microphone_Condenser
- added MK1: CMA-4544PF-W, CMA-4544PF-W:MIC_CMA-4544PF-W, symbol CMA-4544PF-W:CMA-4544PF-W
- JP2: footprint (none) -> Jumper:SolderJumper-3_P1.3mm_Open_RoundedPad1.0x1.5mm_NumberLabels
- JP3: value MIC GAIN -> ATT : REL; footprint (none) -> Jumper:SolderJumper-3_P1.3mm_Open_RoundedPad1.0x1.5mm_NumberLabels
Connections:
- net at C18.2, R14.2: now also MK1.1
- net at C15.2, C16.2, C17.2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: now also MK1.2
