File: Projects/MorayGlow/docs/KiCad/MorayGlow.kicad_sch (KiCad schematic)
At the start: 24 parts, among them J2 RGB LED, J5 Barrel Jack, Q1 IRLML6344TRPBF, Q2 IRLML6344TRPBF, Q3 IRLML6344TRPBF, SW1 SW_DIP_x01, U1 XIAO-ESP32-S3-Plus-SMD

Commit message: updated schmatic and pcb
Parts:
- Q1, Q2, Q3: footprint IRLML6344TRPBF:TRANS_IRLML6344TRPBF -> Package_TO_SOT_SMD:SOT-23
Changed lines of the file:
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@@
 			)
 		)
-		(property "Footprint" "IRLML6344TRPBF:TRANS_IRLML6344TRPBF"
+		(property "Footprint" "Package_TO_SOT_SMD:SOT-23"
 			(at 199.39 30.48 0)
 			(effects
@@
 			)
 		)
-		(property "Footprint" "IRLML6344TRPBF:TRANS_IRLML6344TRPBF"
+		(property "Footprint" "Package_TO_SOT_SMD:SOT-23"
 			(at 157.48 30.48 0)
 			(effects
@@
 			)
 		)
-		(property "Footprint" "IRLML6344TRPBF:TRANS_IRLML6344TRPBF"
+		(property "Footprint" "Package_TO_SOT_SMD:SOT-23"
 			(at 113.03 30.48 0)
 			(effects
